Commit message: Convert dae to usd

File: tests/data/meshes.urdf (robot description, URDF)
Before this commit: robot meshes, 4 links, 3 joints
Links:
- added link link_two_meshes_dae; visual mesh filename=assets/two_meshes.dae scale=0.6 0.6 0.6
- added link link_two_meshes_triangle_dae; visual mesh filename=assets/two_meshes_triangle.dae scale=0.6 0.6 0.6
- link link_mesh_dae: geometry collision mesh filename=assets/box.dae scale=0.8 0.8 0.8; visual mesh filename=assets/box.dae scale=0.8 0.8 0.8
Joints:
- added joint joint_dae_multiple: type fixed, parent link_mesh_dae, child link_two_meshes_dae, origin xyz=1.5 0 0 rpy=0 0 1.570796
- added joint joint_dae_multiple_triangle: type fixed, parent link_two_meshes_dae, child link_two_meshes_triangle_dae, origin xyz=0 -1.5 0 rpy=0 0 0
- joint joint_dae_dxf: parent link_mesh_dae -> link_two_meshes_triangle_dae
- joint joint_obj_dae: origin xyz=1 0 0 rpy=0 0 0 -> xyz=1.5 0 0 rpy=0 0 0

File: tests/data/test_displayname.urdf (robot description, URDF)
Before this commit: robot test_displayname, 2 links, 1 joints
Links:
- added link link-mesh_dae; visual mesh filename=assets/name_test.dae scale=0.5 0.5 0.5
Joints:
- added joint mesh_dae: type fixed, parent link-box2, child link-mesh_dae, origin xyz=0 1 0 rpy=0 0 0
